File: design/PTXXXX_boardname.sch (KiCad schematic (older format))
At the start: 0 parts

Commit message: add text for 1.0 1A release
Other:
- note added: "Add text for 1.0 1A release"
Changed lines of the file:
@@
 Comment4 ""
 $EndDescr
+Text Notes 4750 3900 0    50   ~ 0
+Add text for 1.0 1A release
 $EndSCHEMATC
